File: X15-Backplane.sch (EAGLE design)
At the start: 35 parts

Commit message: Backplane
Other:
- note added: "12V Capacitors"
- note added: "CAN Debug"
- note added: "CAN io"
- note added: "Data Conversion Connector"
- note added: "Dist-Backplane_Logic"
- note added: "Distribution to backplane"
- note added: "Programming"
- note added: "Pwer to ESC adapters"
- note added: "Reset Diode"
- note added: "Solenoid"
- moved on the sheet: C1, C2, C3, C4, C5, C6, CAN_DEBUG, D1, D2, D3, D4, DIST_TO_BACKPLANE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

Commit message: Backplane
Parts:
- removed 7.4V_TO_BACKPLANE: IPL1-104-01-X-S-K, IPL1-104-01-X-S-K:IPL1-104-01-X-S-K
- removed BPK_TO_ROBOT_ARM: IPL1-103-01-L-S-K, IPL1-103-01-L-S-K:IPL1-103-01-L-S-K
- added J1: IPL1-103-01-L-S-K, CONN, Backplane to Robot Arm, IPL1-103-01-L-S-K:IPL1-103-01-L-S-K
- added J2: IPL1-104-01-X-S-K, CONN, 7.4V Power to Backplane, IPL1-104-01-X-S-K:IPL1-104-01-X-S-K
Connections:
- net 7.4V: now also J1.01, J2.01, J2.02; no longer 7.4V_TO_BACKPLANE.01, 7.4V_TO_BACKPLANE.02, BPK_TO_ROBOT_ARM.01
- net 7.4VGND: now also J1.02, J2.03, J2.04; no longer 7.4V_TO_BACKPLANE.03, 7.4V_TO_BACKPLANE.04, BPK_TO_ROBOT_ARM.02
- net ROBOT_ARM: now also J1.03; no longer BPK_TO_ROBOT_ARM.03
Changed lines of the file:
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@@
 <part name="C5" library="CAP, aluminin-capacitor-brick-UCM1H331MNL1GS" deviceset="UCM1H331MNL1GS" device="" package3d_urn="urn:adsk.eagle:package:24202090/2" value="330uF"/>
 <part name="C6" library="CAP, aluminin-capacitor-brick-UCM1H331MNL1GS" deviceset="UCM1H331MNL1GS" device="" package3d_urn="urn:adsk.eagle:package:24202090/2" value="330uF"/>
-<part name="7.4V_TO_BACKPLANE" library="IPL1-104-01-X-S-K" deviceset="IPL1-104-01-X-S-K" device=""/>
 <part name="C7" library="CAP, aluminin-capacitor-brick-UCM1H331MNL1GS" deviceset="UCM1H331MNL1GS" device="" package3d_urn="urn:adsk.eagle:package:24202090/2" value="330uF"/>
 <part name="C8" library="CAP, aluminin-capacitor-brick-UCM1H331MNL1GS" deviceset="UCM1H331MNL1GS" device="" package3d_urn="urn:adsk.eagle:package:24202090/2" value="330uF"/>
@@
 <part name="D5" library="SparkFun-LED" library_urn="urn:adsk.eagle:library:529" deviceset="LED" device="3MM" package3d_urn="urn:adsk.eagle:package:39361/1"/>
 <part name="R1" library="SparkFun-Resistors" library_urn="urn:adsk.eagle:library:532" deviceset="RESISTOR" device="0603" package3d_urn="urn:adsk.eagle:package:39650/1" value="1500"/>
-<part name="BPK_TO_ROBOT_ARM" library="IPL1-103-01-L-S-K" deviceset="IPL1-103-01-L-S-K" device=""/>
 <part name="PI_SHIELD_CONN" library="X15-Pi-Shield-Parts" deviceset="8X_CONN" device=""/>
+<part name="J1" library="CONN, Backplane to Robot Arm, IPL1-103-01-L-S-K" deviceset="IPL1-103-01-L-S-K" device=""/>
+<part name="J2" library="CONN, 7.4V Power to Backplane, IPL1-104-01-X-S-K" deviceset="IPL1-104-01-X-S-K" device=""/>
 </parts>
 <sheets>
@@
 <text x="154.94" y="177.8" size="1.778" layer="91">7.4V Coupling Capacitor</text>
 <text x="48.26" y="78.74" size="1.778" layer="91">Pi Shield Conn</text>
-<text x="68.58" y="137.16" size="1.778" layer="91">BKP to Robot Arm Connector</text>
-<text x="71.12" y="175.26" size="1.778" layer="91">7.4V Power to BKP</text>
+<text x="33.02" y="170.18" size="1.778" layer="91">BKP to Robot Arm Connector</text>
+<text x="33.02" y="134.62" size="1.778" layer="91">7.4V Power to BKP</text>
 <text x="25.4" y="325.12" size="1.778" layer="91">Programming</text>
 <text x="218.44" y="309.88" size="1.778" layer="91">Distribution to backplane</text>
@@
 <attribute name="VALUE" x="260.35" y="237.49" size="1.778" layer="95" align="center-left"/>
 </instance>
-<instance part="7.4V_TO_BACKPLANE" gate="G$1" x="78.74" y="160.02" smashed="yes">
-<attribute name="NAME" x="73.16" y="167.64" size="1.778" layer="95"/>
-<attribute name="VALUE" x="73.66" y="152.4" size="1.778" layer="96"/>
-</instance>
 <instance part="C7" gate="G$1" x="149.86" y="162.56" smashed="yes">
 <attribute name="NAME" x="151.13" y="163.83" size="1.778" layer="95" align="center-left"/>
@@
 <attribute name="VALUE" x="227.076" y="127" size="1.778" layer="96" font="vector" rot="R270" align="top-center"/>
 </instance>
-<instance part="BPK_TO_ROBOT_ARM" gate="G$1" x="78.74" y="127" smashed="yes">
-<attribute name="NAME" x="73.66" y="133.35" size="1.778" layer="95"/>
-<attribute name="VALUE" x="73.66" y="119.38" size="1.778" layer="96"/>
-</instance>
 <instance part="PI_SHIELD_CONN" gate="G$1" x="53.34" y="63.5" smashed="yes">
 <attribute name="NAME" x="48.895" y="73.025" size="1.778" layer="95" font="vector"/>
+</instance>
+<instance part="J1" gate="G$1" x="45.72" y="160.02" smashed="yes">
+<attribute name="NAME" x="40.64" y="166.37" size="1.778" layer="95"/>
+<attribute name="VALUE" x="40.64" y="152.4" size="1.778" layer="96"/>
+</instance>
+<instance part="J2" gate="G$1" x="40.64" y="121.92" smashed="yes">
+<attribute name="NAME" x="35.06" y="129.54" size="1.778" layer="95"/>
+<attribute name="VALUE" x="35.56" y="114.3" size="1.778" layer="96"/>
 </instance>
 </instances>
@@
 <net name="7.4V" class="0">
 <segment>
-<pinref part="7.4V_TO_BACKPLANE" gate="G$1" pin="02"/>
-<pinref part="7.4V_TO_BACKPLANE" gate="G$1" pin="01"/>
-<wire x1="68.58" y1="162.56" x2="68.58" y2="165.1" width="0.1524" layer="91"/>
-<wire x1="68.58" y1="165.1" x2="68.58" y2="170.18" width="0.1524" layer="91"/>
-<junction x="68.58" y="165.1"/>
-<label x="68.58" y="170.18" size="1.778" layer="95"/>
-</segment>
-<segment>
 <pinref part="C7" gate="G$1" pin="+"/>
 <pinref part="C8" gate="G$1" pin="+"/>
@@
 </segment>
 <segment>
-<pinref part="BPK_TO_ROBOT_ARM" gate="G$1" pin="01"/>
-<wire x1="68.58" y1="129.54" x2="55.88" y2="129.54" width="0.1524" layer="91"/>
-<label x="58.42" y="129.54" size="1.778" layer="95"/>
+<pinref part="J1" gate="G$1" pin="01"/>
+<wire x1="35.56" y1="162.56" x2="22.86" y2="162.56" width="0.1524" layer="91"/>
+<label x="25.4" y="162.56" size="1.778" layer="95"/>
+</segment>
+<segment>
+<pinref part="J2" gate="G$1" pin="02"/>
+<pinref part="J2" gate="G$1" pin="01"/>
+<wire x1="30.48" y1="124.46" x2="30.48" y2="127" width="0.1524" layer="91"/>
+<wire x1="30.48" y1="127" x2="30.48" y2="132.08" width="0.1524" layer="91"/>
+<junction x="30.48" y="127"/>
+<label x="30.48" y="132.08" size="1.778" layer="95"/>
 </segment>
 </net>
 <net name="7.4VGND" class="0">
-<segment>
-<pinref part="7.4V_TO_BACKPLANE" gate="G$1" pin="03"/>
-<pinref part="7.4V_TO_BACKPLANE" gate="G$1" pin="04"/>
-<wire x1="68.58" y1="160.02" x2="68.58" y2="157.48" width="0.1524" layer="91"/>
-<wire x1="68.58" y1="157.48" x2="68.58" y2="149.86" width="0.1524" layer="91"/>
-<junction x="68.58" y="157.48"/>
-<label x="68.58" y="149.86" size="1.778" layer="95"/>
-</segment>
 <segment>
 <pinref part="C7" gate="G$1" pin="-"/>
@@
 </segment>
 <segment>
-<pinref part="BPK_TO_ROBOT_ARM" gate="G$1" pin="02"/>
-<wire x1="68.58" y1="127" x2="55.88" y2="127" width="0.1524" layer="91"/>
-<label x="58.42" y="127" size="1.778" layer="95"/>
+<pinref part="J1" gate="G$1" pin="02"/>
+<wire x1="35.56" y1="160.02" x2="22.86" y2="160.02" width="0.1524" layer="91"/>
+<label x="25.4" y="160.02" size="1.778" layer="95"/>
+</segment>
+<segment>
+<pinref part="J2" gate="G$1" pin="03"/>
+<pinref part="J2" gate="G$1" pin="04"/>
+<wire x1="30.48" y1="121.92" x2="30.48" y2="119.38" width="0.1524" layer="91"/>
+<wire x1="30.48" y1="119.38" x2="30.48" y2="114.3" width="0.1524" layer="91"/>
+<junction x="30.48" y="119.38"/>
+<label x="22.86" y="114.3" size="1.778" layer="95"/>
 </segment>
 </net>
@@
 </segment>
 <segment>
-<pinref part="BPK_TO_ROBOT_ARM" gate="G$1" pin="03"/>
-<wire x1="68.58" y1="124.46" x2="55.88" y2="124.46" width="0.1524" layer="91"/>
-<label x="58.42" y="124.46" size="1.778" layer="95"/>
-</segment>
-</net>
+<pinref part="J1" gate="G$1" pin="03"/>
+<wire x1="35.56" y1="157.48" x2="22.86" y2="157.48" width="0.1524" layer="91"/>
+<label x="25.4" y="157.48" size="1.778" layer="95"/>
+</segment>
+</net>

Commit message: Two Sheets
Parts:
- removed C7, C8, C9: 330uF, CAP, aluminin-capacitor-brick-UCM1H331MNL1GS:UCM1H331MNL1GS
- removed D5: (no value), SparkFun-LED:LED3MM
- removed ESC_CONTROL: BACKPLANE_CONNECTORSBKP, Conn, Backplane-ESC-Controller:BACKPLANE_CONNECTORSBKP
- removed J1: IPL1-103-01-L-S-K, CONN, Backplane to Robot Arm, IPL1-103-01-L-S-K:IPL1-103-01-L-S-K
- removed J2: IPL1-104-01-X-S-K, CONN, 7.4V Power to Backplane, IPL1-104-01-X-S-K:IPL1-104-01-X-S-K
- removed PI_SHIELD_CONN: 8X_CONN, X15-Pi-Shield-Parts:8X_CONN
- removed R1: 1500, SparkFun-Resistors:RESISTOR0603
- added C10, C11, C12: 330uF, CAP, aluminin-capacitor-brick-UCM1H331MNL1GS:UCM1H331MNL1GS
- added D6: (no value), SparkFun-LED:LED3MM
- added ESC_CONTROL1: BACKPLANE_CONNECTORSBKP, Conn, Backplane-ESC-Controller:BACKPLANE_CONNECTORSBKP
- added J3: IPL1-103-01-L-S-K, CONN, Backplane to Robot Arm, IPL1-103-01-L-S-K:IPL1-103-01-L-S-K
- added J4: IPL1-104-01-X-S-K, CONN, 7.4V Power to Backplane, IPL1-104-01-X-S-K:IPL1-104-01-X-S-K
- added PI_SHIELD_CONN1: 8X_CONN, X15-Pi-Shield-Parts:8X_CONN
- added R2: 1500, SparkFun-Resistors:RESISTOR0603
Connections:
- removed net N$2: D5.C, R1.1
- new net N$1: D6.C, R2.1
- net 12V: now also PI_SHIELD_CONN1.13, PI_SHIELD_CONN1.15; no longer PI_SHIELD_CONN.13, PI_SHIELD_CONN.15
- net 3V3: now also ESC_CONTROL1.1, ESC_CONTROL1.2, ESC_CONTROL1.3, ESC_CONTROL1.4, PI_SHIELD_CONN1.23; no longer ESC_CONTROL.1, ESC_CONTROL.2, ESC_CONTROL.3, ESC_CONTROL.4, PI_SHIELD_CONN.23
- net 5V: now also PI_SHIELD_CONN1.19; no longer PI_SHIELD_CONN.19
- net 7.4V: now also C10.+, C11.+, C12.+, D6.A, J3.01, J4.01, J4.02; no longer C7.+, C8.+, C9.+, D5.A, J1.01, J2.01, J2.02
- net 7.4VGND: now also C10.-, C11.-, C12.-, J3.02, J4.03, J4.04, R2.2; no longer C7.-, C8.-, C9.-, J1.02, J2.03, J2.04, R1.2
- net CAN_H: now also ESC_CONTROL1.5, PI_SHIELD_CONN1.1; no longer ESC_CONTROL.5, PI_SHIELD_CONN.1
- net CAN_L: now also ESC_CONTROL1.7, PI_SHIELD_CONN1.2; no longer ESC_CONTROL.7, PI_SHIELD_CONN.2
- net ESC_ID: now also ESC_CONTROL1.12; no longer ESC_CONTROL.12
- net GND: now also ESC_CONTROL1.10, PI_SHIELD_CONN1.17, PI_SHIELD_CONN1.21; no longer ESC_CONTROL.10, PI_SHIELD_CONN.17, PI_SHIELD_CONN.21
- net NRST: now also ESC_CONTROL1.6; no longer ESC_CONTROL.6
- net ROBOT_ARM: now also J3.03, PI_SHIELD_CONN1.4; no longer J1.03, PI_SHIELD_CONN.4
- net SOL1_1: now also PI_SHIELD_CONN1.14; no longer PI_SHIELD_CONN.14
- net SOL2_1: now also PI_SHIELD_CONN1.16; no longer PI_SHIELD_CONN.16
- net SOL3_1: now also PI_SHIELD_CONN1.18; no longer PI_SHIELD_CONN.18
- net SOL4_1: now also PI_SHIELD_CONN1.20; no longer PI_SHIELD_CONN.20
- net SOL5_1: now also PI_SHIELD_CONN1.22; no longer PI_SHIELD_CONN.22
- net SOL6_1: now also PI_SHIELD_CONN1.24; no longer PI_SHIELD_CONN.24
- net SWCLK: now also ESC_CONTROL1.11; no longer ESC_CONTROL.11
- net SWDIO: now also ESC_CONTROL1.9; no longer ESC_CONTROL.9

Commit message: Two Sheets
Parts:
- C10, C11, C12, C2, C3, C4, C5, C6: device CAP, aluminin-capacitor-brick-UCM1H331MNL1GS:UCM1H331MNL1GS -> X15-Backplane Parts:UCM1H331MNL1GS
- CAN_DEBUG: device CONN, Phoenix Contact PTSM-04-V-1778573:PXC-PTSM-04-RA-1778641 -> X15-Backplane Parts:PXC-PTSM-04-RA-1778641
- DIST_TO_BACKPLANE: device CONN, Samtec MPPT Hermaphoditic 10 pos - MPPT-10-01-01-L-RA-SD:MPPT-10-01-01-L-RA-SD -> X15-Backplane Parts:MPPT-10-01-01-L-RA-SD
- ESC_CONTROL1: device Conn, Backplane-ESC-Controller:BACKPLANE_CONNECTORSBKP -> X15-Backplane Parts:BACKPLANE_CONNECTORSBKP
- H1, H2: device OTHER, Mounting Holes:6-32-HOLE -> X15-Backplane Parts:6-32-HOLE
- J3: device CONN, Backplane to Robot Arm, IPL1-103-01-L-S-K:IPL1-103-01-L-S-K -> X15-Backplane Parts:IPL1-103-01-L-S-K
- J4: device CONN, 7.4V Power to Backplane, IPL1-104-01-X-S-K:IPL1-104-01-X-S-K -> X15-Backplane Parts:IPL1-104-01-X-S-K
- MUX: device IC, 4to1 BackplaneMUX:TI-SN74LV4052A -> X15-Backplane Parts:TI-SN74LV4052A
- PI_SHIELD_CONN1: device X15-Pi-Shield-Parts:8X_CONN -> X15-Backplane Parts:8X_CONN
- PXC-8-RA-1, PXC-8-RA-1778683: device CONN, Phoenix Contact PTSM 8 pin:PXC-8-RA-1778683 -> X15-Backplane Parts:PXC-8-RA-1778683
- U$4, U$5, U$6: device CONN, Backplane_ESC_adapter:BACKPLANE_ESC_ADAPTER_PWRBKP -> X15-Backplane Parts:BACKPLANE_ESC_ADAPTER_PWRBKP
- U$7: device OTHER, Push button - FSM2JMTR:DISCRETECOMPONENTS_SWITCH -> X15-Backplane Parts:DISCRETECOMPONENTS_SWITCH
- U$8: device CONN, Distribution-Backplane:BACKPLANE-DISTRIBUTION -> X15-Backplane Parts:BACKPLANE-DISTRIBUTION
- U$9: device CONN, DataConversion-Backplane Connector- SAMTEC CLT-107-01-F-D:BACKPLANE->DATACONV -> X15-Backplane Parts:BACKPLANE->DATACONV
Changed lines of the file:
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@@
 <parts>
 <part name="FRAME2" library="SparkFun-Aesthetics" library_urn="urn:adsk.eagle:library:507" deviceset="FRAME-A4L" device=""/>
-<part name="MUX" library="IC, 4to1 BackplaneMUX" deviceset="TI-SN74LV4052A" device=""/>
-<part name="PXC-8-RA-1778683" library="CONN, Phoenix Contact PTSM 8 pin" deviceset="PXC-8-RA-1778683" device="" package3d_urn="urn:adsk.eagle:package:25224885/2">
+<part name="MUX" library="X15-Backplane Parts" deviceset="TI-SN74LV4052A" device=""/>
+<part name="PXC-8-RA-1778683" library="X15-Backplane Parts" deviceset="PXC-8-RA-1778683" device="" package3d_urn="urn:adsk.eagle:package:25224885/2">
 <attribute name="SPICEPREFIX" value="X"/>
 </part>
-<part name="U$4" library="CONN, Backplane_ESC_adapter" deviceset="BACKPLANE_ESC_ADAPTER_PWR" device="BKP"/>
-<part name="U$5" library="CONN, Backplane_ESC_adapter" deviceset="BACKPLANE_ESC_ADAPTER_PWR" device="BKP"/>
-<part name="U$6" library="CONN, Backplane_ESC_adapter" deviceset="BACKPLANE_ESC_ADAPTER_PWR" device="BKP"/>
-<part name="PXC-8-RA-1" library="CONN, Phoenix Contact PTSM 8 pin" deviceset="PXC-8-RA-1778683" device="" package3d_urn="urn:adsk.eagle:package:25224885/2">
+<part name="U$4" library="X15-Backplane Parts" deviceset="BACKPLANE_ESC_ADAPTER_PWR" device="BKP"/>
+<part name="U$5" library="X15-Backplane Parts" deviceset="BACKPLANE_ESC_ADAPTER_PWR" device="BKP"/>
+<part name="U$6" library="X15-Backplane Parts" deviceset="BACKPLANE_ESC_ADAPTER_PWR" device="BKP"/>
+<part name="PXC-8-RA-1" library="X15-Backplane Parts" deviceset="PXC-8-RA-1778683" device="" package3d_urn="urn:adsk.eagle:package:25224885/2">
 <attribute name="SPICEPREFIX" value="X"/>
 </part>
@@
 <part name="D3" library="SparkFun-DiscreteSemi" library_urn="urn:adsk.eagle:library:514" deviceset="DIODE-SCHOTTKY" device="-PMEG4005EJ" package3d_urn="urn:adsk.eagle:package:38441/1" value="0.5A/40V/420mV"/>
 <part name="D4" library="SparkFun-DiscreteSemi" library_urn="urn:adsk.eagle:library:514" deviceset="DIODE-SCHOTTKY" device="-PMEG4005EJ" package3d_urn="urn:adsk.eagle:package:38441/1" value="0.5A/40V/420mV"/>
-<part name="U$7" library="OTHER, Push button - FSM2JMTR" deviceset="DISCRETECOMPONENTS_SWITCH" device="" package3d_urn="urn:adsk.eagle:package:24384574/2"/>
+<part name="U$7" library="X15-Backplane Parts" deviceset="DISCRETECOMPONENTS_SWITCH" device="" package3d_urn="urn:adsk.eagle:package:24384574/2"/>
 <part name="R4" library="SparkFun-Resistors" library_urn="urn:adsk.eagle:library:532" deviceset="RESISTOR" device="0603" package3d_urn="urn:adsk.eagle:package:39650/1" value="10k"/>
-<part name="DIST_TO_BACKPLANE" library="CONN, Samtec MPPT Hermaphoditic 10 pos - MPPT-10-01-01-L-RA-SD" deviceset="MPPT-10-01-01-L-RA-SD" device="" package3d_urn="urn:adsk.eagle:package:25115828/2"/>
-<part name="U$8" library="CONN, Distribution-Backplane" deviceset="BACKPLANE-DISTRIBUTION" device=""/>
-<part name="H1" library="OTHER, Mounting Holes" deviceset="6-32-HOLE" device="" package3d_urn="urn:adsk.eagle:package:24384748/2"/>
-<part name="H2" library="OTHER, Mounting Holes" deviceset="6-32-HOLE" device="" package3d_urn="urn:adsk.eagle:package:24384748/2"/>
-<part name="CAN_DEBUG" library="CONN, Phoenix Contact PTSM-04-V-1778573" deviceset="PXC-PTSM-04-RA-1778641" device=""/>
+<part name="DIST_TO_BACKPLANE" library="X15-Backplane Parts" deviceset="MPPT-10-01-01-L-RA-SD" device="" package3d_urn="urn:adsk.eagle:package:25115828/2"/>
+<part name="U$8" library="X15-Backplane Parts" deviceset="BACKPLANE-DISTRIBUTION" device=""/>
+<part name="H1" library="X15-Backplane Parts" deviceset="6-32-HOLE" device="" package3d_urn="urn:adsk.eagle:package:24384748/2"/>
+<part name="H2" library="X15-Backplane Parts" deviceset="6-32-HOLE" device="" package3d_urn="urn:adsk.eagle:package:24384748/2"/>
+<part name="CAN_DEBUG" library="X15-Backplane Parts" deviceset="PXC-PTSM-04-RA-1778641" device=""/>
 <part name="R5" library="SparkFun-Resistors" library_urn="urn:adsk.eagle:library:532" deviceset="RESISTOR" device="0603" package3d_urn="urn:adsk.eagle:package:39650/1" value="60"/>
 <part name="R6" library="SparkFun-Resistors" library_urn="urn:adsk.eagle:library:532" deviceset="RESISTOR" device="0603" package3d_urn="urn:adsk.eagle:package:39650/1" value="60"/>
 <part name="C1" library="SparkFun-Capacitors" library_urn="urn:adsk.eagle:library:510" deviceset="0.1UF" device="-0603-100V-10%" package3d_urn="urn:adsk.eagle:package:37414/1" value="0.1uF"/>
-<part name="U$9" library="CONN, DataConversion-Backplane Connector- SAMTEC CLT-107-01-F-D" deviceset="BACKPLANE-&gt;DATACONV" device=""/>
-<part name="C2" library="CAP, aluminin-capacitor-brick-UCM1H331MNL1GS" deviceset="UCM1H331MNL1GS" device="" package3d_urn="urn:adsk.eagle:package:24202090/2" value="330uF"/>
-<part name="C3" library="CAP, aluminin-capacitor-brick-UCM1H331MNL1GS" deviceset="UCM1H331MNL1GS" device="" package3d_urn="urn:adsk.eagle:package:24202090/2" value="330uF"/>
-<part name="C4" library="CAP, aluminin-capacitor-brick-UCM1H331MNL1GS" deviceset="UCM1H331MNL1GS" device="" package3d_urn="urn:adsk.eagle:package:24202090/2" value="330uF"/>
-<part name="C5" library="CAP, aluminin-capacitor-brick-UCM1H331MNL1GS" deviceset="UCM1H331MNL1GS" device="" package3d_urn="urn:adsk.eagle:package:24202090/2" value="330uF"/>
-<part name="C6" library="CAP, aluminin-capacitor-brick-UCM1H331MNL1GS" deviceset="UCM1H331MNL1GS" device="" package3d_urn="urn:adsk.eagle:package:24202090/2" value="330uF"/>
+<part name="U$9" library="X15-Backplane Parts" deviceset="BACKPLANE-&gt;DATACONV" device=""/>
+<part name="C2" library="X15-Backplane Parts" deviceset="UCM1H331MNL1GS" device="" package3d_urn="urn:adsk.eagle:package:24202090/2" value="330uF"/>
+<part name="C3" library="X15-Backplane Parts" deviceset="UCM1H331MNL1GS" device="" package3d_urn="urn:adsk.eagle:package:24202090/2" value="330uF"/>
+<part name="C4" library="X15-Backplane Parts" deviceset="UCM1H331MNL1GS" device="" package3d_urn="urn:adsk.eagle:package:24202090/2" value="330uF"/>
+<part name="C5" library="X15-Backplane Parts" deviceset="UCM1H331MNL1GS" device="" package3d_urn="urn:adsk.eagle:package:24202090/2" value="330uF"/>
+<part name="C6" library="X15-Backplane Parts" deviceset="UCM1H331MNL1GS" device="" package3d_urn="urn:adsk.eagle:package:24202090/2" value="330uF"/>
 <part name="FRAME3" library="SparkFun-Aesthetics" library_urn="urn:adsk.eagle:library:507" deviceset="FRAME-A4L" device=""/>
-<part name="C10" library="CAP, aluminin-capacitor-brick-UCM1H331MNL1GS" deviceset="UCM1H331MNL1GS" device="" package3d_urn="urn:adsk.eagle:package:24202090/2" value="330uF"/>
-<part name="C11" library="CAP, aluminin-capacitor-brick-UCM1H331MNL1GS" deviceset="UCM1H331MNL1GS" device="" package3d_urn="urn:adsk.eagle:package:24202090/2" value="330uF"/>
-<part name="C12" library="CAP, aluminin-capacitor-brick-UCM1H331MNL1GS" deviceset="UCM1H331MNL1GS" device="" package3d_urn="urn:adsk.eagle:package:24202090/2" value="330uF"/>
-<part name="ESC_CONTROL1" library="Conn, Backplane-ESC-Controller" deviceset="BACKPLANE_CONNECTORS" device="BKP"/>
+<part name="C10" library="X15-Backplane Parts" deviceset="UCM1H331MNL1GS" device="" package3d_urn="urn:adsk.eagle:package:24202090/2" value="330uF"/>
+<part name="C11" library="X15-Backplane Parts" deviceset="UCM1H331MNL1GS" device="" package3d_urn="urn:adsk.eagle:package:24202090/2" value="330uF"/>
+<part name="C12" library="X15-Backplane Parts" deviceset="UCM1H331MNL1GS" device="" package3d_urn="urn:adsk.eagle:package:24202090/2" value="330uF"/>
+<part name="ESC_CONTROL1" library="X15-Backplane Parts" deviceset="BACKPLANE_CONNECTORS" device="BKP"/>
 <part name="D6" library="SparkFun-LED" library_urn="urn:adsk.eagle:library:529" deviceset="LED" device="3MM" package3d_urn="urn:adsk.eagle:package:39361/1"/>
 <part name="R2" library="SparkFun-Resistors" library_urn="urn:adsk.eagle:library:532" deviceset="RESISTOR" device="0603" package3d_urn="urn:adsk.eagle:package:39650/1" value="1500"/>
-<part name="PI_SHIELD_CONN1" library="X15-Pi-Shield-Parts" deviceset="8X_CONN" device=""/>
-<part name="J3" library="CONN, Backplane to Robot Arm, IPL1-103-01-L-S-K" deviceset="IPL1-103-01-L-S-K" device=""/>
-<part name="J4" library="CONN, 7.4V Power to Backplane, IPL1-104-01-X-S-K" deviceset="IPL1-104-01-X-S-K" device=""/>
+<part name="PI_SHIELD_CONN1" library="X15-Backplane Parts" deviceset="8X_CONN" device=""/>
+<part name="J3" library="X15-Backplane Parts" deviceset="IPL1-103-01-L-S-K" device=""/>
+<part name="J4" library="X15-Backplane Parts" deviceset="IPL1-104-01-X-S-K" device=""/>
 </parts>
 <sheets>
