File: X15-Backplane.brd (EAGLE design)
At the start: 139.7 x 100 mm, 31 parts, among them U1 ULN2003AD

Commit message: ESC Fixed
Parts:
- moved ESC_CONTROLLER 24.4 mm to (80.5, 7.62)
- moved C6 20.3 mm to (48.8, 13.0)
- moved C5 15.0 mm to (37.6, 13.0)
- moved D7 13.7 mm to (111.5, 3.05)
- moved R3 13.7 mm to (113.3, 9.14)
- moved R6 1.63 mm to (45.5, 75.2)
Routing:
- net 3V3: track 272.0 -> 307.0 mm
- net CAN_H: track 277.8 -> 302.0 mm
- net CAN_L: track 265.9 -> 289.9 mm
- net N$4: track 14.6 -> 16.1 mm
- net 7.4V: track 146.8 -> 147.3 mm
